File: TestRevA/TestA.sch (EAGLE design)
At the start: 51 parts, among them IC1 SI7021, IC2 ATMEGA328-PB, IC3 PE4259, IC4 NCS7SZ04, U1 V_REG_317SMD, U2 LSM9DS1, Y1 16MHz, Y2 16MHz

Commit message: Finished schematic
Got rid of UHF inverter, changed all components to 0402 from 0603, made DIO connections.
Parts:
- removed IC4: NCS7SZ04, Mini-Project:NCS7SZ04
- removed Q1: (no value), crystal-geyer_V1_0:KXO-TCXO-CMOS-86
- removed R6: nc, SparkFun:RESISTOR0603-RES
- removed R7: 360, SparkFun:RESISTOR0603-RES
- removed R9: 100, SparkFun:RESISTOR0603-RES
- added C27: 47pF, SparkFun:CAP0402-CAP
- added C28: 1nF, SparkFun:CAP0402-CAP
- added C29, C31: nc, SparkFun:CAP0402-CAP
- added ISP1: AVRISP-6, adafruit:AVRISP-6
- added SW1: (no value), adafruit:SWITCH_PUSHBUTTONSOFTTOUCHSMD_SJ
- C1: value 0.1 uF -> 26pF; device SparkFun:CAP0603-CAP -> SparkFun:CAP0402-CAP
- C10: value 0.1uF -> 10uF; device SparkFun:CAP0603-CAP -> SparkFun:CAP0402-CAP
- C11: value 10uF -> 10pF; device SparkFun:CAP0603-CAP -> SparkFun:CAP0402-CAP
- C12, C18: device SparkFun:CAP0603-CAP -> SparkFun:CAP0402-CAP
- C13: value 26pF -> 10nF; device SparkFun:CAP0603-CAP -> SparkFun:CAP0402-CAP
- C14: value 26pF -> 0.1uF; device SparkFun:CAP0603-CAP -> SparkFun:CAP0402-CAP
- C15: value 4.7pF -> 100nF; device SparkFun:CAP0603-CAP -> SparkFun:CAP0402-CAP
- C16: value 1.8pF -> 47pF; device SparkFun:CAP0603-CAP -> SparkFun:CAP0402-CAP
- C17: value 47pF -> 1.5pF; device SparkFun:CAP0603-CAP -> SparkFun:CAP0402-CAP
- C19: value nc -> 33pF; device SparkFun:CAP0603-CAP -> SparkFun:CAP0402-CAP
- C2: value nc -> 26pF; device SparkFun:CAP0603-CAP -> SparkFun:CAP0402-CAP
- C20: value 1nF -> 10nF; device SparkFun:CAP0603-CAP -> SparkFun:CAP0402-CAP
- C21: value 1nF -> 3.3pF; device SparkFun:CAP0603-CAP -> SparkFun:CAP0402-CAP
- C22: value 100nF -> 4.7pF; device SparkFun:CAP0603-CAP -> SparkFun:CAP0402-CAP
- C23: value 47pF -> 1.2pF; device SparkFun:CAP0603-CAP -> SparkFun:CAP0402-CAP
- C24: value 10nF -> 47pF; device SparkFun:CAP0603-CAP -> SparkFun:CAP0402-CAP
- C25: value 100nF -> 1.8pF; device SparkFun:CAP0603-CAP -> SparkFun:CAP0402-CAP
- C3: value 3.3pF -> 0.1 uF; device SparkFun:CAP0603-CAP -> SparkFun:CAP0402-CAP
- C4: value 47pF -> 1uF; device SparkFun:CAP0603-CAP -> SparkFun:CAP0402-CAP
- C5: value 33pF -> 0.1uF; device SparkFun:CAP0603-CAP -> SparkFun:CAP0402-CAP
- C6: value 1.5pF -> 10pF; device SparkFun:CAP0603-CAP -> SparkFun:CAP0402-CAP
- C7: value 1.2pF -> 100nF; device SparkFun:CAP0603-CAP -> SparkFun:CAP0402-CAP
- C8: value 10nF -> 100nF; device SparkFun:CAP0603-CAP -> SparkFun:CAP0402-CAP
- C9: value 0.1uF -> 100nF; device SparkFun:CAP0603-CAP -> SparkFun:CAP0402-CAP
- L1: value 10nF -> nc; device SparkFun:INDUCTOR0603 -> SparkFun:INDUCTOR0402
- L2: value 10nH -> 10nF; device SparkFun:INDUCTOR0603 -> SparkFun:INDUCTOR0402
- L3: value 6.2nH -> 10nH; device SparkFun:INDUCTOR0603 -> SparkFun:INDUCTOR0402
- L4: value 0R -> 6.2nH; device SparkFun:INDUCTOR0603 -> SparkFun:INDUCTOR0402
- L5: value nc -> 0R; device SparkFun:INDUCTOR0603 -> SparkFun:INDUCTOR0402
- R1, R2: device SparkFun:RESISTOR0603-RES -> SparkFun:RESISTOR0402-RES
- R3: value 10K -> 220; device SparkFun:RESISTOR0603-RES -> SparkFun:RESISTOR0402-RES
- R4: value 220 -> 360; device SparkFun:RESISTOR0603-RES -> SparkFun:RESISTOR0402-RES
- R5: value 0 -> 10K; device SparkFun:RESISTOR0603-RES -> SparkFun:RESISTOR0402-RES
- R8: value nc -> 0; device SparkFun:RESISTOR0603-RES -> SparkFun:RESISTOR0402-RES
- Y2: value 16MHz -> 32Mhz
- renumbered RF2 to RF1
Connections:
- removed net N$19: C20.1, IC3.CTRL, IC4.Y, R6.2
- removed net N$20: C22.2, IC4.VCC
- removed net N$21: IC4.A, R6.1, R8.2, R9.2
- removed net RXTXEXT: R8.1
- new net DIO0: IC2.PD6(OC0A/PTCXY/AIN0), RF1.DIO0
- new net DIO1: IC2.PD7(ICP1/CLKO/PTCXY), RF1.DIO1
- new net DIO2: IC2.PB0(ICP1/CLKO/PTCXY), RF1.DIO2
- new net DIO3: IC2.PB1(OC1A/PTCXY), RF1.DIO3
- new net N$23: IC2.PC1(ADC1/PTCY/SCK1), ISP1.SCK
- new net N$24: C7.1, RF1.VR_ANA
- new net N$25: C9.1, RF1.VR_DIG
- new net N$26: IC2.PC0(ADC0/PTCY/MISO1), ISP1.MISO
- new net N$27: IC2.PE3(ADC7/PTCY/T3/MOSI1), ISP1.MOSI
- new net XTA: C6.1, RF1.XTA, Y2.1
- new net XTB: C11.1, RF1.XTB, Y2.2
- net +3.3V: now also C10.1, C15.1, C28.1, C3.1, C5.1, C8.1, ISP1.VCC, R1.1, R5.2, RF1.VBAT1; no longer C1.1, C11.1, C12.1, C21.1, C25.1, R1.2, R3.1
- net 3.3V: now also C4.1, R3.2; no longer R4.2
- net GND: now also C17.2, C22.2, C28.2, C29.2, C31.2, C4.2, C5.2, C7.2, ISP1.GND, R4.1, SW1.P$2; no longer C19.2, C22.1, C23.2, C24.2, IC4.GND, R7.1
- net I1: now also IC2.PD2(PTCXY/INT0/OC3B/OC4B); no longer IC2.PC6(RST)
- net N$1: now also C24.1, R8.2; no longer C4.1, R5.2
- net N$10: now also C21.1, L2.2, R8.1; no longer C3.1, L1.2, R5.1
- net N$11: now also C17.1, C19.1, L1.1; no longer C5.1, C6.1, L5.1
- net N$12: now also C22.1, C23.1, L3.2, L4.1; no longer C15.1, C7.1, L2.2, L3.1
- net N$13: now also C19.2, L3.1; no longer C5.2, L2.1
- net N$14: now also C23.2, C25.1, IC3.RF1, L4.2; no longer C16.1, C7.2, IC3.RF2, L3.2
- net N$15: now also C31.1, L5.2; no longer C19.1, L4.2
- net N$16: now also C27.1; no longer C17.1
- net N$17: now also C14.1; no longer C9.1
- net N$18: now also C27.2, C29.1, L5.1; no longer C17.2, C18.1, L4.1
- net N$2: now also C16.1, C20.1, L1.2; no longer C23.1, C24.1, L5.2
- net N$22: now also IC2.PC6(RST), ISP1.RST, SW1.P$1; no longer RF1.RST
- net N$4: now also C24.2, IC3.RF2; no longer C4.2, IC3.RF1
- net N$5: now also R5.1; no longer R1.1
- net N$6: now also R3.1, R4.2; no longer R4.1, R7.2
- net N$7: now also C18.1, L2.1; no longer C2.1, L1.1
- net N$8: now also C13.1; no longer C8.1
- net N$9: now also C12.1; no longer C10.1
- net RXTXX: now also IC3.CTRL; no longer R9.1
- net SCL: now also R1.2; no longer R2.2
- net SDA: now also R2.2; no longer R3.2
- net XTAL1: now also C1.1; no longer C14.1
- net XTAL2: now also C2.1; no longer C13.1
Other:
- moved on the sheet: C1, C10, C11, C12, C13, C14, C15, C16, C17, C18, C19, C2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

Commit message: Completed board design, DRC and finishing touches remaining
Connections:
- removed net SS: RF1.NSS
- new net DIO4: IC2.PD5(OC0B/T1/PTCXY), RF1.DIO4
- new net DIO5: IC2.PE2(ADC6/PTCY/ICP3/SS1), RF1.DIO5
- net DIO0: now also IC2.PB1(OC1A/PTCXY); no longer IC2.PD6(OC0A/PTCXY/AIN0)
- net DIO1: now also IC2.PB0(ICP1/CLKO/PTCXY); no longer IC2.PD7(ICP1/CLKO/PTCXY)
- net DIO2: now also IC2.PD7(ICP1/CLKO/PTCXY); no longer IC2.PB0(ICP1/CLKO/PTCXY)
- net DIO3: now also IC2.PD6(OC0A/PTCXY/AIN0); no longer IC2.PB1(OC1A/PTCXY)
- net EN: now also RF1.NSS
- net I1: now also U2.DRDY_M; no longer U2.INT1_A/G
- net I2: now also IC2.PC3(ADC3/PTCY); no longer IC2.PE2(ADC6/PTCY/ICP3/SS1)
- net I3: now also U2.INT_M; no longer U2.DRDY_M
- net I4: now also U2.INT1_A/G; no longer U2.INT_M
Changed lines of the file:
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@@
 <label x="27.94" y="12.7" size="1.778" layer="95" rot="R180" xref="yes"/>
 </segment>
+<segment>
+<pinref part="RF1" gate="G$1" pin="NSS"/>
+<wire x1="213.36" y1="35.56" x2="215.9" y2="35.56" width="0.1524" layer="91"/>
+<label x="215.9" y="35.56" size="1.778" layer="95" xref="yes"/>
+</segment>
 </net>
 <net name="I1" class="0">
-<segment>
-<pinref part="U2" gate="G$1" pin="INT1_A/G"/>
-<wire x1="226.06" y1="116.84" x2="228.6" y2="116.84" width="0.1524" layer="91"/>
-<label x="228.6" y="116.84" size="1.778" layer="95" xref="yes"/>
-</segment>
 <segment>
 <label x="104.14" y="78.74" size="1.778" layer="95" xref="yes"/>
@@
 <wire x1="104.14" y1="78.74" x2="99.06" y2="78.74" width="0.1524" layer="91"/>
 </segment>
+<segment>
+<pinref part="U2" gate="G$1" pin="DRDY_M"/>
+<wire x1="228.6" y1="106.68" x2="226.06" y2="106.68" width="0.1524" layer="91"/>
+<label x="228.6" y="106.68" size="1.778" layer="95" xref="yes"/>
+</segment>
 </net>
 <net name="I2" class="0">
@@
 </segment>
 <segment>
-<label x="104.14" y="12.7" size="1.778" layer="95" xref="yes"/>
-<pinref part="IC2" gate="G$1" pin="PE2(ADC6/PTCY/ICP3/SS1)"/>
-<wire x1="104.14" y1="12.7" x2="99.06" y2="12.7" width="0.1524" layer="91"/>
+<label x="104.14" y="48.26" size="1.778" layer="95" xref="yes"/>
+<pinref part="IC2" gate="G$1" pin="PC3(ADC3/PTCY)"/>
+<wire x1="104.14" y1="48.26" x2="99.06" y2="48.26" width="0.1524" layer="91"/>
 </segment>
 </net>
 <net name="I3" class="0">
-<segment>
-<pinref part="U2" gate="G$1" pin="DRDY_M"/>
-<wire x1="226.06" y1="106.68" x2="231.14" y2="106.68" width="0.1524" layer="91"/>
-<label x="231.14" y="106.68" size="1.778" layer="95" xref="yes"/>
-</segment>
 <segment>
 <label x="104.14" y="73.66" size="1.778" layer="95" xref="yes"/>
@@
 <wire x1="99.06" y1="73.66" x2="104.14" y2="73.66" width="0.1524" layer="91"/>
 </segment>
-</net>
-<net name="I4" class="0">
 <segment>
 <pinref part="U2" gate="G$1" pin="INT_M"/>
@@
 <label x="236.22" y="104.14" size="1.778" layer="95" xref="yes"/>
 </segment>
+</net>
+<net name="I4" class="0">
 <segment>
 <label x="104.14" y="68.58" size="1.778" layer="95" xref="yes"/>
 <pinref part="IC2" gate="G$1" pin="PD0(PTCXY/OC3A/RXD0)"/>
 <wire x1="99.06" y1="68.58" x2="104.14" y2="68.58" width="0.1524" layer="91"/>
+</segment>
+<segment>
+<label x="228.6" y="116.84" size="1.778" layer="95" xref="yes"/>
+<pinref part="U2" gate="G$1" pin="INT1_A/G"/>
+<wire x1="228.6" y1="116.84" x2="226.06" y2="116.84" width="0.1524" layer="91"/>
 </segment>
 </net>
@@
 <wire x1="86.36" y1="109.22" x2="86.36" y2="111.76" width="0.1524" layer="91"/>
 <junction x="86.36" y="111.76"/>
-</segment>
-</net>
-<net name="SS" class="0">
-<segment>
-<pinref part="RF1" gate="G$1" pin="NSS"/>
-<wire x1="213.36" y1="35.56" x2="215.9" y2="35.56" width="0.1524" layer="91"/>
-<label x="215.9" y="35.56" size="1.778" layer="95" xref="yes"/>
 </segment>
 </net>
@@
 <net name="DIO1" class="0">
 <segment>
+<pinref part="IC2" gate="G$1" pin="PB0(ICP1/CLKO/PTCXY)"/>
+<wire x1="33.02" y1="22.86" x2="30.48" y2="22.86" width="0.1524" layer="91"/>
+<label x="30.48" y="22.86" size="1.778" layer="95" rot="R180" xref="yes"/>
+</segment>
+<segment>
 <pinref part="RF1" gate="G$1" pin="DIO1"/>
 <wire x1="172.72" y1="30.48" x2="167.64" y2="30.48" width="0.1524" layer="91"/>
 <label x="167.64" y="30.48" size="1.778" layer="95" rot="R180" xref="yes"/>
 </segment>
+</net>
+<net name="DIO0" class="0">
+<segment>
+<pinref part="IC2" gate="G$1" pin="PB1(OC1A/PTCXY)"/>
+<wire x1="33.02" y1="17.78" x2="30.48" y2="17.78" width="0.1524" layer="91"/>
+<label x="30.48" y="17.78" size="1.778" layer="95" rot="R180" xref="yes"/>
+</segment>
+<segment>
+<pinref part="RF1" gate="G$1" pin="DIO0"/>
+<wire x1="172.72" y1="35.56" x2="167.64" y2="35.56" width="0.1524" layer="91"/>
+<label x="167.64" y="35.56" size="1.778" layer="95" rot="R180" xref="yes"/>
+</segment>
+</net>
+<net name="DIO2" class="0">
 <segment>
 <pinref part="IC2" gate="G$1" pin="PD7(ICP1/CLKO/PTCXY)"/>
@@
 <label x="30.48" y="27.94" size="1.778" layer="95" rot="R180" xref="yes"/>
 </segment>
-</net>
-<net name="DIO0" class="0">
+<segment>
+<pinref part="RF1" gate="G$1" pin="DIO2"/>
+<wire x1="172.72" y1="25.4" x2="167.64" y2="25.4" width="0.1524" layer="91"/>
+<label x="167.64" y="25.4" size="1.778" layer="95" rot="R180" xref="yes"/>
+</segment>
+</net>
+<net name="DIO3" class="0">
 <segment>
 <pinref part="IC2" gate="G$1" pin="PD6(OC0A/PTCXY/AIN0)"/>
 <wire x1="33.02" y1="33.02" x2="30.48" y2="33.02" width="0.1524" layer="91"/>
 <label x="30.48" y="33.02" size="1.778" layer="95" rot="R180" xref="yes"/>
-</segment>
-<segment>
-<pinref part="RF1" gate="G$1" pin="DIO0"/>
-<wire x1="172.72" y1="35.56" x2="167.64" y2="35.56" width="0.1524" layer="91"/>
-<label x="167.64" y="35.56" size="1.778" layer="95" rot="R180" xref="yes"/>
-</segment>
-</net>
-<net name="DIO2" class="0">
-<segment>
-<pinref part="IC2" gate="G$1" pin="PB0(ICP1/CLKO/PTCXY)"/>
-<wire x1="33.02" y1="22.86" x2="30.48" y2="22.86" width="0.1524" layer="91"/>
-<label x="30.48" y="22.86" size="1.778" layer="95" rot="R180" xref="yes"/>
-</segment>
-<segment>
-<pinref part="RF1" gate="G$1" pin="DIO2"/>
-<wire x1="172.72" y1="25.4" x2="167.64" y2="25.4" width="0.1524" layer="91"/>
-<label x="167.64" y="25.4" size="1.778" layer="95" rot="R180" xref="yes"/>
-</segment>
-</net>
-<net name="DIO3" class="0">
-<segment>
-<pinref part="IC2" gate="G$1" pin="PB1(OC1A/PTCXY)"/>
-<wire x1="33.02" y1="17.78" x2="30.48" y2="17.78" width="0.1524" layer="91"/>
-<label x="30.48" y="17.78" size="1.778" layer="95" rot="R180" xref="yes"/>
 </segment>
 <segment>
@@
 </segment>
 </net>
+<net name="DIO4" class="0">
+<segment>
+<pinref part="IC2" gate="G$1" pin="PD5(OC0B/T1/PTCXY)"/>
+<wire x1="33.02" y1="38.1" x2="30.48" y2="38.1" width="0.1524" layer="91"/>
+<label x="30.48" y="38.1" size="1.778" layer="95" rot="R180" xref="yes"/>
+</segment>
+<segment>
+<pinref part="RF1" gate="G$1" pin="DIO4"/>
+<wire x1="172.72" y1="15.24" x2="167.64" y2="15.24" width="0.1524" layer="91"/>
+<label x="167.64" y="15.24" size="1.778" layer="95" rot="R180" xref="yes"/>
+</segment>
+</net>
+<net name="DIO5" class="0">
+<segment>
+<pinref part="IC2" gate="G$1" pin="PE2(ADC6/PTCY/ICP3/SS1)"/>
+<wire x1="99.06" y1="12.7" x2="104.14" y2="12.7" width="0.1524" layer="91"/>
+<label x="104.14" y="12.7" size="1.778" layer="95" xref="yes"/>
+</segment>
+<segment>
+<pinref part="RF1" gate="G$1" pin="DIO5"/>
+<wire x1="172.72" y1="10.16" x2="167.64" y2="10.16" width="0.1524" layer="91"/>
+<label x="167.64" y="10.16" size="1.778" layer="95" rot="R180" xref="yes"/>
+</segment>
+</net>
